Commit message: joint space locked

File: src/feeding_deployment/robot_controller/hack_gen3_robotiq_2f_85.urdf (robot description, URDF)
Before this commit: robot gen3_robotiq_2f_85, 11 links, 10 joints
Links:
- link robotiq_arg2f_base_link: mass 1.6 -> 0.9
Joints:
- joint joint_6: origin xyz=0 0.00017505 -0.10593 rpy=1.5708 9.2076E-28 -8.2157E-15 -> xyz=0 0.00017505 -0.10593 rpy=1.5708 1.18051646 -8.2157E-15; type revolute -> fixed
