Commit message: drink transfer

File: src/feeding_deployment/robot_controller/hack_gen3_robotiq_2f_85_drink.urdf (robot description, URDF)
Before this commit: robot gen3_robotiq_2f_85_feeding, 14 links, 13 joints
Links:
- link robotiq_arg2f_base_link: mass 1.0 -> 1.7

Commit message: tuned task space controller to be less jerky + full drink

File: src/feeding_deployment/robot_controller/hack_gen3_robotiq_2f_85_drink.urdf (robot description, URDF)
Before this commit: robot gen3_robotiq_2f_85_feeding, 14 links, 13 joints
Links:
- link robotiq_arg2f_base_link: mass 1.7 -> 2.0

File: src/feeding_deployment/robot_controller/hack_gen3_robotiq_2f_85_wipe.urdf (robot description, URDF)
Before this commit: robot gen3_robotiq_2f_85_feeding, 14 links, 13 joints
Links:
- link robotiq_arg2f_base_link: mass 1.0 -> 1.3

Commit message: tuned new values for fork and empty drink

File: src/feeding_deployment/robot_controller/hack_gen3_robotiq_2f_85_drink.urdf (robot description, URDF)
Before this commit: robot gen3_robotiq_2f_85_feeding, 14 links, 13 joints
Links:
- link robotiq_arg2f_base_link: mass 2.0 -> 1.9

File: src/feeding_deployment/robot_controller/hack_gen3_robotiq_2f_85_fork.urdf (robot description, URDF)
Before this commit: robot gen3_robotiq_2f_85_feeding, 17 links, 16 joints
Links:
- link robotiq_arg2f_base_link: mass 1.7 -> 1.5
