Commit message: propagated drink utensil calibration to task space compliant controllers

File: src/feeding_deployment/robot_controller/hack_gen3_robotiq_2f_85_drink_10_5.urdf (robot description, URDF)
Before this commit: robot gen3_robotiq_2f_85_feeding, 14 links, 13 joints
Joints:
- joint joint_drink_tip: origin xyz=0.27 0.095 -0.045 rpy=0 1.570796 0 -> xyz=0.22 0.03 -0.037 rpy=0 1.570796 0

File: src/feeding_deployment/robot_controller/hack_gen3_robotiq_2f_85_drink_12.urdf (robot description, URDF)
Before this commit: robot gen3_robotiq_2f_85_feeding, 14 links, 13 joints
Joints:
- joint joint_drink_tip: origin xyz=0.27 0.095 -0.045 rpy=0 1.570796 0 -> xyz=0.22 0.03 -0.037 rpy=0 1.570796 0

File: src/feeding_deployment/robot_controller/hack_gen3_robotiq_2f_85_drink_6.urdf (robot description, URDF)
Before this commit: robot gen3_robotiq_2f_85_feeding, 14 links, 13 joints
Joints:
- joint joint_drink_tip: origin xyz=0.27 0.095 -0.045 rpy=0 1.570796 0 -> xyz=0.22 0.03 -0.037 rpy=0 1.570796 0

File: src/feeding_deployment/robot_controller/hack_gen3_robotiq_2f_85_drink_7_5.urdf (robot description, URDF)
Before this commit: robot gen3_robotiq_2f_85_feeding, 14 links, 13 joints
Joints:
- joint joint_drink_tip: origin xyz=0.27 0.095 -0.045 rpy=0 1.570796 0 -> xyz=0.22 0.03 -0.037 rpy=0 1.570796 0

File: src/feeding_deployment/robot_controller/hack_gen3_robotiq_2f_85_drink_9.urdf (robot description, URDF)
Before this commit: robot gen3_robotiq_2f_85_feeding, 14 links, 13 joints
Joints:
- joint joint_drink_tip: origin xyz=0.27 0.095 -0.045 rpy=0 1.570796 0 -> xyz=0.22 0.03 -0.037 rpy=0 1.570796 0

Commit message: calibrated final drink tip

File: src/feeding_deployment/robot_controller/hack_gen3_robotiq_2f_85_drink_10_5.urdf (robot description, URDF)
Before this commit: robot gen3_robotiq_2f_85_feeding, 14 links, 13 joints
Joints:
- joint joint_drink_tip: origin xyz=0.22 0.03 -0.037 rpy=0 1.570796 0 -> xyz=0.21 0.07 -0.037 rpy=0 1.570796 0

File: src/feeding_deployment/robot_controller/hack_gen3_robotiq_2f_85_drink_12.urdf (robot description, URDF)
Before this commit: robot gen3_robotiq_2f_85_feeding, 14 links, 13 joints
Joints:
- joint joint_drink_tip: origin xyz=0.22 0.03 -0.037 rpy=0 1.570796 0 -> xyz=0.21 0.07 -0.037 rpy=0 1.570796 0

File: src/feeding_deployment/robot_controller/hack_gen3_robotiq_2f_85_drink_6.urdf (robot description, URDF)
Before this commit: robot gen3_robotiq_2f_85_feeding, 14 links, 13 joints
Joints:
- joint joint_drink_tip: origin xyz=0.22 0.03 -0.037 rpy=0 1.570796 0 -> xyz=0.21 0.07 -0.037 rpy=0 1.570796 0

File: src/feeding_deployment/robot_controller/hack_gen3_robotiq_2f_85_drink_7_5.urdf (robot description, URDF)
Before this commit: robot gen3_robotiq_2f_85_feeding, 14 links, 13 joints
Joints:
- joint joint_drink_tip: origin xyz=0.22 0.03 -0.037 rpy=0 1.570796 0 -> xyz=0.21 0.07 -0.037 rpy=0 1.570796 0

File: src/feeding_deployment/robot_controller/hack_gen3_robotiq_2f_85_drink_9.urdf (robot description, URDF)
Before this commit: robot gen3_robotiq_2f_85_feeding, 14 links, 13 joints
Joints:
- joint joint_drink_tip: origin xyz=0.22 0.03 -0.037 rpy=0 1.570796 0 -> xyz=0.21 0.07 -0.037 rpy=0 1.570796 0
