Commit message: outside-mouth transfer seems to work in sim

File: src/feeding_deployment/assets/urdf/feeding_utensil/feeding_utensil.urdf (robot description, URDF)
Before this commit: robot feeding_utensil, 5 links, 4 joints
Links:
- link forkbase: geometry visual mesh filename=utensil_base.stl
- link forkpitch: geometry visual mesh filename=pitch_link.stl
- link forkroll: geometry visual mesh filename=roll_link.stl
