Commit message: utensil pickup -> acq (without FLAIR) -> transfer in sim

File: src/feeding_deployment/assets/urdf/drinking_utensil/drinking_utensil.urdf (robot description, URDF)
Before this commit: robot drinking_utensil, 1 links, 0 joints
Links:
- link drinkbase: geometry visual mesh filename=utensil_base.stl

File: src/feeding_deployment/assets/urdf/wiping_utensil/wiping_utensil.urdf (robot description, URDF)
Before this commit: robot wiping_utensil, 1 links, 0 joints
Links:
- link wipebase: geometry visual mesh filename=utensil_base.stl
