Commit message: editing tool masses

File: src/feeding_deployment/robot_controller/urdfs/hack_gen3_robotiq_2f_85_fork.urdf (robot description, URDF)
Before this commit: robot gen3_robotiq_2f_85_feeding, 17 links, 16 joints
Links:
- link robotiq_arg2f_base_link: mass 1.5 -> 1.6

File: src/feeding_deployment/robot_controller/urdfs/hack_gen3_robotiq_2f_85_wipe.urdf (robot description, URDF)
Before this commit: robot gen3_robotiq_2f_85_feeding, 14 links, 13 joints
Links:
- link robotiq_arg2f_base_link: mass 1.3 -> 1.6

Commit message: pre-pilot edits

File: src/feeding_deployment/robot_controller/urdfs/hack_gen3_robotiq_2f_85_fork.urdf (robot description, URDF)
Before this commit: robot gen3_robotiq_2f_85_feeding, 17 links, 16 joints
Links:
- link robotiq_arg2f_base_link: mass 1.6 -> 1.5
