Commit message: cleanup

File: src/feeding_deployment/assets/wheelchair/wheelchair.urdf (robot description, URDF)
Before this commit: robot wheelchair, 1 links, 0 joints
Links:
- link base_link: geometry collision mesh filename=simplified_wheelchair.obj scale=1 1 1; visual mesh filename=wheelchair.obj scale=1 1 1
