Commit message: drinking utensil model + pose fixed

File: src/feeding_deployment/assets/drinking_utensil/drinking_utensil.urdf (robot description, URDF)
Before this commit: robot drinking_utensil, 1 links, 0 joints
Links:
- link drinkbase: geometry visual mesh filename=mug_with_holder.obj

File: src/feeding_deployment/assets/table/table.urdf (robot description, URDF)
Before this commit: robot table, 1 links, 0 joints
Links:
- link table: geometry collision mesh filename=simplified_table.obj; visual mesh filename=table_new.obj
