Commit message: checked errors for different states

File: src/feeding_deployment/control/robot_controller/urdfs/gen3_robotiq_2f_85_drink.urdf (robot description, URDF)
Before this commit: robot gen3_robotiq_2f_85, 11 links, 10 joints
Links:
- added link drink_tip, mass 0
- added link drinkbase, mass 0; collision mesh filename=package://kortex_description/tools/drinking_tool/tool_base.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; visual mesh filename=package://kortex_description/tools/drinking_tool/tool_base.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
- added link finger_tip, mass 0
- link end_effector_link: mass None -> 0
- link robotiq_arg2f_base_link: mass 0.9 -> 1.9
- link tool_frame: mass None -> 0
Joints:
- added joint finger_tip_joint: type fixed, parent end_effector_link, child finger_tip, origin xyz=0 0 0.17955 rpy=0 0 0
- added joint finger_tip_to_drinkbase: type fixed, parent finger_tip, child drinkbase, origin xyz=0 0 0 rpy=0 0 0
- added joint joint_drink_tip: type fixed, parent drinkbase, child drink_tip, origin xyz=0.21 0.07 -0.037 rpy=0 1.570796 0, axis 0 0 0, limit lower=0 upper=0 effort=2000 velocity=1
- joint end_effector: axis 0 0 0 -> (none)
- joint tool_frame_joint: axis 0 0 0 -> (none)

File: src/feeding_deployment/control/robot_controller/urdfs/gen3_robotiq_2f_85_fork.urdf (robot description, URDF)
Before this commit: robot gen3_robotiq_2f_85, 11 links, 10 joints
Links:
- added link feeding_tool_tip, mass 0
- added link finger_tip, mass 0
- added link fork_tip, mass 0
- added link forkbase, mass 0; collision mesh filename=package://kortex_description/tools/feeding_tool/tool_base.s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; visual mesh filename=package://kortex_description/tools/feeding_tool/tool_base.s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
- added link forkpitch, mass 0; collision mesh filename=package://kortex_description/tools/feeding_tool/tool_pitch.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; visual mesh filename=package://kortex_description/tools/feeding_tool/tool_pitch.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
- added link forkroll, mass 0; collision mesh filename=package://kortex_description/tools/feeding_tool/tool_roll.s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; visual mesh filename=package://kortex_description/tools/feeding_tool/tool_roll.s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
- link end_effector_link: mass None -> 0
- link robotiq_arg2f_base_link: mass 0.9 -> 1.5
- link tool_frame: mass None -> 0
Joints:
- added joint finger_tip_joint: type fixed, parent end_effector_link, child finger_tip, origin xyz=0 0 0.17955 rpy=0 0 0
- added joint finger_tip_to_forkbase: type fixed, parent finger_tip, child forkbase, origin xyz=0 0 0 rpy=0 0 0
- added joint forkpitch_joint: type fixed, parent forkbase, child forkpitch, origin xyz=0.11 0.0 -0.087 rpy=0 0 0
- added joint forkroll_joint: type fixed, parent forkpitch, child forkroll, origin xyz=0.0151 0.0 0.0095   rpy=-1.570796 0 0
- added joint joint_feeding_tool_tip: type fixed, parent forkroll, child feeding_tool_tip, origin xyz=0.13 0.0 0.003 rpy=0 0 0
- added joint joint_fork_tip: type fixed, parent feeding_tool_tip, child fork_tip, origin xyz=0.0 0 0.0 rpy=1.570796 0 1.570796
- joint end_effector: axis 0 0 0 -> (none)
- joint tool_frame_joint: axis 0 0 0 -> (none)

File: src/feeding_deployment/control/robot_controller/urdfs/gen3_robotiq_2f_85_wipe.urdf (robot description, URDF)
Before this commit: robot gen3_robotiq_2f_85, 11 links, 10 joints
Links:
- added link finger_tip, mass 0
- added link wipe_tip, mass 0
- added link wipebase, mass 0; collision mesh filename=package://kortex_description/tools/wiping_tool/tool_base.stl; visual mesh filename=package://kortex_description/tools/wiping_tool/tool_base.stl
- link end_effector_link: mass None -> 0
- link robotiq_arg2f_base_link: mass 0.9 -> 1.3
- link tool_frame: mass None -> 0
Joints:
- added joint finger_tip_joint: type fixed, parent end_effector_link, child finger_tip, origin xyz=0 0 0.17955 rpy=0 0 0
- added joint finger_tip_to_wipebase: type fixed, parent finger_tip, child wipebase, origin xyz=0 0 0 rpy=0 0 0
- added joint joint_wip_tip: type fixed, parent wipebase, child wipe_tip, origin xyz=0.089 -0.015 -0.078 rpy=0 1.570796 0
- joint end_effector: axis 0 0 0 -> (none)
- joint tool_frame_joint: axis 0 0 0 -> (none)
