Commit message: updated fork urdf - controller tuning

File: src/feeding_deployment/control/robot_controller/urdfs/hack_gen3_robotiq_2f_85_fork.urdf (robot description, URDF)
Before this commit: robot gen3_robotiq_2f_85_feeding, 17 links, 16 joints
Links:
- link robotiq_arg2f_base_link: mass 1.5 -> 1.3

Commit message: [nuc] tested bite / sip / wipe transfer for Benjamin's head pose

File: src/feeding_deployment/control/robot_controller/urdfs/hack_gen3_robotiq_2f_85_fork.urdf (robot description, URDF)
Before this commit: robot gen3_robotiq_2f_85_feeding, 17 links, 16 joints
Links:
- link robotiq_arg2f_base_link: mass 1.3 -> 1.5
