Commit message: cleaned up local workspace and editing wiping tool length

File: src/feeding_deployment/control/robot_controller/urdfs/gen3_robotiq_2f_85_wipe.urdf (robot description, URDF)
Before this commit: robot gen3_robotiq_2f_85_feeding, 14 links, 13 joints
Joints:
- joint joint_wip_tip: origin xyz=0.089 -0.015 -0.078 rpy=0 1.570796 0 -> xyz=0.139 -0.015 -0.078 rpy=0 1.570796 0

File: src/feeding_deployment/control/robot_controller/urdfs/hack_gen3_robotiq_2f_85_wipe.urdf (robot description, URDF)
Before this commit: robot gen3_robotiq_2f_85_feeding, 14 links, 13 joints
Joints:
- joint joint_wip_tip: origin xyz=0.089 -0.015 -0.078 rpy=0 1.570796 0 -> xyz=0.139 -0.015 -0.078 rpy=0 1.570796 0
